File: Calculatrix.kicad_sch (KiCad schematic)
At the start: 96 parts, among them J1 +5V, Q1 MMBT3904, SW1 7, SW10 2, SW11 3, SW12 -, SW13 0, SW14 ., SW15 ±, SW16 +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

Commit message: clean up
Parts:
- D24: value Ready/Busy -> Busy/Ready
Changed lines of the file:
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@@
 			)
 		)
-		(property "Value" "Ready/Busy"
+		(property "Value" "Busy/Ready"
 			(at 391.9347 148.59 0)
 			(show_name no)
